File: CM5IO.kicad_pcb (KiCad board)
At the start: 4 copper layers, 56 parts, among them J1 DF17_1.0H_-80DP-0.5V_57_, J11 USB_C_Receptacle_USB2.0, J14 JST_SHBM04B-SRSS-TB, J2 Conn_02x07_Odd_Even, J22 690-019-298-412, J3 Conn_01x03, J4 Bus_M.2_Socket_M, J5 USB3_A, J8 THD-20-R, SW1 Right angle Tact button, U12 RT9742SNGV, U5 74LVC1G07SE-7, U6 AP22653W6, U7 ASEK-32.768KHZ-L-R-T, U8 AP3441SHE-7B

Commit message: PCB Layout edited
Parts:
- added H5: MountingHole, CM5IO:MountingHole_2.7mm_M2.5_DIN965, F.Cu at (106.8, 106.8)
- added H6: MountingHole, CM5IO:MountingHole_2.7mm_M2.5_DIN965, F.Cu at (106.8, 113.1)
- added H7: MountingHole, CM5IO:MountingHole_2.7mm_M2.5_DIN965, F.Cu at (106.8, 119.3)
- added H8: MountingHole, CM5IO:MountingHole_2.7mm_M2.5_DIN965, F.Cu at (106.8, 125.6)
- added J6: Conn_01x06_Socket, Connector_Molex:Molex_MicroClasp_55932-0630_1x06_P2.00mm_Vertical, F.Cu at (116.0, 108.5)
- added J7: Conn_01x06_Socket, Connector_Molex:Molex_MicroClasp_55932-0630_1x06_P2.00mm_Vertical, F.Cu at (116.0, 117.2)
Connections:
- J1 pad 1: unconnected-(J1-Pad1) -> FMU-SWDIO
- J1 pad 10: unconnected-(J1-Pad10) -> CAN_H_3
- J1 pad 11: unconnected-(J1-Pad11) -> EXTERN_DRDY
- J1 pad 12: unconnected-(J1-Pad12) -> SERIAL5 RX
- J1 pad 13: unconnected-(J1-Pad13) -> GND
- J1 pad 14: unconnected-(J1-Pad14) -> SERIAL5 TX
- J1 pad 15: unconnected-(J1-Pad15) -> GND
- J1 pad 16: unconnected-(J1-Pad16) -> SERIAL4 RX
- J1 pad 17: unconnected-(J1-Pad17) -> SAFETY
- J1 pad 18: unconnected-(J1-Pad18) -> SERIAL4 TX
- J1 pad 19: unconnected-(J1-Pad19) -> VDD 3V3 SPEKTRUM EN
- J1 pad 2: unconnected-(J1-Pad2) -> ~{FMU-LED AMBER}
- J1 pad 20: unconnected-(J1-Pad20) -> SERIAL3 RX
- J1 pad 21: unconnected-(J1-Pad21) -> PRESSURE SENS IN
- J1 pad 22: unconnected-(J1-Pad22) -> SERIAL3 TX
- J1 pad 23: unconnected-(J1-Pad23) -> AUX BATT VOLTAGE SENS
- J1 pad 24: unconnected-(J1-Pad24) -> ALARM
- J1 pad 25: unconnected-(J1-Pad25) -> AUX BATT CURRENT SENS
- J1 pad 27: unconnected-(J1-Pad27) -> ~{VDD 5V PERIPH EN}
- J1 pad 28: unconnected-(J1-Pad28) -> ~{IO-LED SAFET PROT}
- J1 pad 29: unconnected-(J1-Pad29) -> VBUS
- J1 pad 3: unconnected-(J1-Pad3) -> FMU-SWCLK
- J1 pad 30: unconnected-(J1-Pad30) -> SERIAL2 RTS
- J1 pad 31: unconnected-(J1-Pad31) -> OTG_DP1
- J1 pad 32: unconnected-(J1-Pad32) -> SERIAL2 CTS
- J1 pad 33: unconnected-(J1-Pad33) -> OTG_DM1
- J1 pad 34: unconnected-(J1-Pad34) -> SERIAL2 RX
- J1 pad 35: unconnected-(J1-Pad35) -> I2C_1_SDA
- J1 pad 36: unconnected-(J1-Pad36) -> SERIAL2 TX
- J1 pad 37: unconnected-(J1-Pad37) -> I2C_1_SCL
- J1 pad 38: unconnected-(J1-Pad38) -> SERIAL 1 RX
- J1 pad 39: unconnected-(J1-Pad39) -> CAN_L_2
- J1 pad 4: unconnected-(J1-Pad4) -> I2C_2_SDA
- J1 pad 40: unconnected-(J1-Pad40) -> SERIAL1 TX
- J1 pad 41: unconnected-(J1-Pad41) -> CAN_H_2
- J1 pad 42: unconnected-(J1-Pad42) -> SERIAL1 RTS
- J1 pad 43: unconnected-(J1-Pad43) -> ~{VDD 5V PERIPH OC}
- J1 pad 44: unconnected-(J1-Pad44) -> SERIAL1 CTS
- J1 pad 45: unconnected-(J1-Pad45) -> ~{VDD 5V HIPOWER OC}
- J1 pad 46: unconnected-(J1-Pad46) -> IO-USART1 TX
- J1 pad 47: unconnected-(J1-Pad47) -> BATT VOLTAGE PROT
- J1 pad 48: unconnected-(J1-Pad48) -> IO-USART1 RX SPECTRUM_DSM
- J1 pad 49: unconnected-(J1-Pad49) -> BATT CURRENT SENS PROT
- J1 pad 5: unconnected-(J1-Pad5) -> ~{EXTERN CS}
- J1 pad 50: unconnected-(J1-Pad50) -> FMU-CH1-PROT
- J1 pad 51: unconnected-(J1-Pad51) -> SPI_EXT_MOSI
- J1 pad 52: unconnected-(J1-Pad52) -> FMU-CH2-PROT
- J1 pad 53: unconnected-(J1-Pad53) -> VDD SERVO
- J1 pad 54: unconnected-(J1-Pad54) -> FMU-CH3-PROT
- J1 pad 55: unconnected-(J1-Pad55) -> ~{VDD BRICK VALID}
- J1 pad 56: unconnected-(J1-Pad56) -> FMU-CH4-PROT
- J1 pad 57: unconnected-(J1-Pad57) -> ~{VDD BACKUP VALID}
- J1 pad 58: unconnected-(J1-Pad58) -> FMU-CH5-PROT
- J1 pad 59: unconnected-(J1-Pad59) -> ~{VBUS VALID}
- J1 pad 6: unconnected-(J1-Pad6) -> I2C_2_SDA
- J1 pad 60: unconnected-(J1-Pad60) -> FMU-CH6-PROT
- J1 pad 61: unconnected-(J1-Pad61) -> VDD 5V IN PROT
- J1 pad 62: unconnected-(J1-Pad62) -> PPM-SBUS-PROT
- J1 pad 63: unconnected-(J1-Pad63) -> VDD 5V IN PROT
- J1 pad 64: unconnected-(J1-Pad64) -> S.BUS OUT
- J1 pad 66: unconnected-(J1-Pad66) -> IO-CH8-PROT
- J1 pad 67: unconnected-(J1-Pad67) -> SPI_EXT_MISO
- J1 pad 68: unconnected-(J1-Pad68) -> IO-CH7-PROT
- J1 pad 69: unconnected-(J1-Pad69) -> IO-SWDIO
- J1 pad 7: unconnected-(J1-Pad7) -> FMU-!RESET
- J1 pad 70: unconnected-(J1-Pad70) -> IO-CH6-PROT
- J1 pad 71: unconnected-(J1-Pad71) -> IO-SWCLK
- J1 pad 72: unconnected-(J1-Pad72) -> IO-CH5-PROT
- J1 pad 73: unconnected-(J1-Pad73) -> SPI_EXT_SCK
- J1 pad 74: unconnected-(J1-Pad74) -> IO-CH4-PROT
- J1 pad 75: unconnected-(J1-Pad75) -> IO-!RESET
- J1 pad 76: unconnected-(J1-Pad76) -> IO-CH3-PROT
- J1 pad 77: unconnected-(J1-Pad77) -> CAN_L_1
- J1 pad 78: unconnected-(J1-Pad78) -> IO-CH2-PROT
- J1 pad 79: unconnected-(J1-Pad79) -> CAN_H_1
- J1 pad 8: unconnected-(J1-Pad8) -> CAN_L_3
- J1 pad 80: unconnected-(J1-Pad80) -> IO-CH1-PROT
- J1 pad 9: unconnected-(J1-Pad9) -> VDD SERVO IN
- PSM1 pad !VBUS_VALID: unconnected-(PSM1-~{VBUS_VALID}-Pad!VBUS_VALID) -> /CM5_GPIO ( Ethernet, GPIO, SDCARD)/Cube_PSM_GPIO/~{VBUS_VALID}
- PSM1 pad !VDD_5V_HIPOWER_OC: unconnected-(PSM1-~{VDD_5V_HIPOWER_OC}-Pad!VDD_5V_HIPOWER_OC) -> /CM5_GPIO ( Ethernet, GPIO, SDCARD)/Cube_PSM_GPIO/~{VDD_5V_HIPOWER_OC}
- PSM1 pad !VDD_5V_PERIPH_EN: unconnected-(PSM1-~{VDD_5V_PERIPH_EN}-Pad!VDD_5V_PERIPH_EN) -> /CM5_GPIO ( Ethernet, GPIO, SDCARD)/Cube_PSM_GPIO/~{VDD_5V_PERIPH_EN}
- PSM1 pad !VDD_5V_PERIPH_OC: unconnected-(PSM1-~{VDD_5V_PERIPH_OC}-Pad!VDD_5V_PERIPH_OC) -> /CM5_GPIO ( Ethernet, GPIO, SDCARD)/Cube_PSM_GPIO/~{VDD_5V_PERIPH_OC}
- PSM1 pad !VDD_BACKUP_VALID: unconnected-(PSM1-~{VDD_BACKUP_VALID}-Pad!VDD_BACKUP_VALID) -> /CM5_GPIO ( Ethernet, GPIO, SDCARD)/Cube_PSM_GPIO/~{VDD_BACKUP_VALID}
- PSM1 pad !VDD_BRICK_VALID: unconnected-(PSM1-~{VDD_BRICK_VALID}-Pad!VDD_BRICK_VALID) -> /CM5_GPIO ( Ethernet, GPIO, SDCARD)/Cube_PSM_GPIO/~{VDD_BRICK_VALID}
- PSM1 pad 5V_HIPOWER: unconnected-(PSM1-VDD_5V_HIPOWER-Pad5V_HIPOWER) -> /CM5_GPIO ( Ethernet, GPIO, SDCARD)/Cube_PSM_GPIO/VDD_5V_HIPOWER
- PSM1 pad 5V_PERIPH: unconnected-(PSM1-VDD_5V_PERIPH-Pad5V_PERIPH) -> /CM5_GPIO ( Ethernet, GPIO, SDCARD)/Cube_PSM_GPIO/VDD_5V_PERIPH
- PSM1 pad ALARM: unconnected-(PSM1-PadALARM) -> ALARM
- PSM1 pad BUZZER_OUT: unconnected-(PSM1-BUZZ_OUT-PadBUZZER_OUT) -> /CM5_GPIO ( Ethernet, GPIO, SDCARD)/Cube_PSM_GPIO/BUZZER_OUT
- PSM1 pad GND: unconnected-(PSM1-PadGND) -> GND
- PSM1 pad RX: unconnected-(PSM1-RX_5V_out-PadRX) -> /CM5_GPIO ( Ethernet, GPIO, SDCARD)/Cube_PSM_GPIO/RX_5v0_OUT
- PSM1 pad SERVO_IN: unconnected-(PSM1-PadSERVO_IN) -> /CM5_GPIO ( Ethernet, GPIO, SDCARD)/Cube_PSM_GPIO/VDD_SERVO_IN
- PSM1 pad SPEK: unconnected-(PSM1-VDD_3V3_SPEKTRUM-PadSPEK) -> /CM5_GPIO ( Ethernet, GPIO, SDCARD)/Cube_PSM_GPIO/VDD_3v3_SPEKTRUM
- PSM1 pad VBUS: unconnected-(PSM1-VBUS_TO_FMU-PadVBUS) -> /CM5_GPIO ( Ethernet, GPIO, SDCARD)/Cube_PSM_GPIO/VBUS_TO_FMU
- PSM1 pad VDD_3V3_SPEKTRUM_EN: unconnected-(PSM1-PadVDD_3V3_SPEKTRUM_EN) -> /CM5_GPIO ( Ethernet, GPIO, SDCARD)/Cube_PSM_GPIO/VDD_3v3_SPEKTRUM_EN
- PSM1 pad VDD_5V_BACKUP: unconnected-(PSM1-PadVDD_5V_BACKUP) -> /CM5_GPIO ( Ethernet, GPIO, SDCARD)/Cube_PSM_GPIO/VDD_5V_BACKUP
- PSM1 pad VDD_5V_IN_PROT: unconnected-(PSM1-VDD_5V_TO_FMU-PadVDD_5V_IN_PROT) -> /CM5_GPIO ( Ethernet, GPIO, SDCARD)/Cube_PSM_GPIO/VDD_5V_IN_PROT
- PSM1 pad VDD_BRICK_IN: unconnected-(PSM1-PadVDD_BRICK_IN) -> /CM5_GPIO ( Ethernet, GPIO, SDCARD)/Cube_PSM_GPIO/VDD_5V_BRICK
- PSM1 pad VDD_VBUS: unconnected-(PSM1-PadVDD_VBUS) -> VBUS
